File: kicad Esp32-ETH/ETH/placa.kicad_pcb (KiCad board)
At the start: 2 copper layers, 4 parts, among them J6 ESP32

Commit message: Listo para Probar
Connections:
- H1 pad 11: RTSN -> unconnected-(H1-RSTN-Pad11)
- H1 pad 6: unconnected-(H1-INTN-Pad6) -> INT
- U3 pad 35: unconnected-(U3-Pad35) -> INT
Routing:
- net INT: track 0.00 -> 78.8 mm
- net RTSN: track 63.8 -> 0.00 mm
- net 5V: track 103.2 -> 61.8 mm
- net VCC: track 74.6 -> 88.3 mm
- net GND: track 131.4 -> 123.9 mm
- net MOSI: track 53.6 -> 51.9 mm
- net CS: track 27.4 -> 28.6 mm
- net SCLK: track 40.1 -> 39.4 mm
